File: open_controler_thermal/thermal/digital.sch (KiCad schematic (older format))
At the start: 54 parts, among them J1 Conn_01x02, J2 Conn_02x20_Odd_Even, J3 e_i_01x10, J4 e_i_02x10, J5 a_i_01x10

Commit message: trabajando en la huella del ESP32
Parts:
- added U?: ESP32_NODEMCU_OS, MODULE_ESP32_NODEMCU, symbol ESP32_NODEMCU:ESP32_NODEMCU_OS
Changed lines of the file:
@@
 Text GLabel 10465 2800 0    50   Input ~ 0
 jG21
+$Comp
+L ESP32_NODEMCU:ESP32_NODEMCU_OS U?
+U 1 1 6323ED7B
+P 12970 1930
+F 0 "U?" H 12970 3297 50  0000 C CNN
+F 1 "ESP32_NODEMCU_OS" H 12970 3206 50  0000 C CNN
+F 2 "MODULE_ESP32_NODEMCU" H 11140 2970 50  0001 L BNN
+F 3 "" H 12970 1930 50  0001 L BNN
+F 4 "Espressif" H 12970 1930 50  0001 L BNN "MANUFACTURER"
+F 5 "6.6 mm" H 11750 3300 50  0001 L BNN "MAXIMUM_PACKAGE_HEIGHT"
+F 6 "Manufacturer Recommendations" H 12540 3310 50  0001 L BNN "STANDARD"
+	1    12970 1930
+	1    0    0    -1
+$EndComp
 $EndSCHEMATC

Commit message: diseñando PCB thermal con ESP32
Parts:
- removed U?: ESP32_NODEMCU_OS, MODULE_ESP32_NODEMCU, symbol ESP32_NODEMCU:ESP32_NODEMCU_OS
- added U?: ESP32_NODEMCU_OS, ESP32, symbol ESP32_NODEMCU:ESP32_NODEMCU_OS
- C10, C11, C12, C13, C14, C15, C16, C17, C18, C19, C2, C3, C4, C5, C6, C7, C8, C9: symbol wat-rescue:C -> digital-rescue:C-wat-rescue
- R1, R10, R11, R12, R13, R14, R15, R16, R17, R18, R19, R2, R20, R21, R22, R23, R24, R25, R26, R27, R28, R3, R4, R5, R6, R7, R8, R9: symbol wat-rescue:R -> digital-rescue:R-wat-rescue
- Uxxx1: symbol wat-rescue:NANO-nano -> digital-rescue:NANO-nano-wat-rescue
Changed lines of the file:
@@
 NoConn ~ 4875 -920
 $Comp
-L wat-rescue:C C2
+L digital-rescue:C-wat-rescue C2
 U 1 1 5FF955E2
 P 1530 3830
@@
 $EndComp
 $Comp
-L wat-rescue:R R7
+L digital-rescue:R-wat-rescue R7
 U 1 1 5FF955F0
 P 1220 3830
@@
 $EndComp
 $Comp
-L wat-rescue:R R1
+L digital-rescue:R-wat-rescue R1
 U 1 1 5FF955F7
 P 930 3610
@@
 	1080 3610 1220 3610
 $Comp
-L wat-rescue:C C8
+L digital-rescue:C-wat-rescue C8
 U 1 1 5FFB1A03
 P 1090 5465
@@
 $EndComp
 $Comp
-L wat-rescue:R R13
+L digital-rescue:R-wat-rescue R13
 U 1 1 5FFB1A2C
 P 1090 5025
@@
 	1090 4875 1090 4695
 $Comp
-L wat-rescue:C C3
+L digital-rescue:C-wat-rescue C3
 U 1 1 5FFCF401
 P 3150 3830
@@
 $EndComp
 $Comp
-L wat-rescue:R R8
+L digital-rescue:R-wat-rescue R8
 U 1 1 5FFCF40F
 P 2840 3830
@@
 $EndComp
 $Comp
-L wat-rescue:R R2
+L digital-rescue:R-wat-rescue R2
 U 1 1 5FFCF416
 P 2550 3610
@@
 	2700 3610 2840 3610
 $Comp
-L wat-rescue:C C4
+L digital-rescue:C-wat-rescue C4
 U 1 1 5FFD4082
 P 4780 3830
@@
 $EndComp
 $Comp
-L wat-rescue:R R9
+L digital-rescue:R-wat-rescue R9
 U 1 1 5FFD4090
 P 4470 3830
@@
 $EndComp
 $Comp
-L wat-rescue:R R3
+L digital-rescue:R-wat-rescue R3
 U 1 1 5FFD4097
 P 4180 3610
@@
 	4330 3610 4470 3610
 $Comp
-L wat-rescue:C C5
+L digital-rescue:C-wat-rescue C5
 U 1 1 5FFD40B3
 P 6490 3830
@@
 $EndComp
 $Comp
-L wat-rescue:R R10
+L digital-rescue:R-wat-rescue R10
 U 1 1 5FFD40C1
 P 6180 3830
@@
 $EndComp
 $Comp
-L wat-rescue:R R4
+L digital-rescue:R-wat-rescue R4
 U 1 1 5FFD40C8
 P 5890 3610
@@
 	6040 3610 6180 3610
 $Comp
-L wat-rescue:C C6
+L digital-rescue:C-wat-rescue C6
 U 1 1 5FFEEFC9
 P 8215 3830
@@
 $EndComp
 $Comp
-L wat-rescue:R R11
+L digital-rescue:R-wat-rescue R11
 U 1 1 5FFEEFD7
 P 7905 3830
@@
 $EndComp
 $Comp
-L wat-rescue:R R5
+L digital-rescue:R-wat-rescue R5
 U 1 1 5FFEEFDE
 P 7615 3610
@@
 	7765 3610 7905 3610
 $Comp
-L wat-rescue:C C7
+L digital-rescue:C-wat-rescue C7
 U 1 1 5FFEEFFA
 P 9835 3830
@@
 $EndComp
 $Comp
-L wat-rescue:R R12
+L digital-rescue:R-wat-rescue R12
 U 1 1 5FFEF008
 P 9525 3830
@@
 $EndComp
 $Comp
-L wat-rescue:R R6
+L digital-rescue:R-wat-rescue R6
 U 1 1 5FFEF00F
 P 9235 3610
@@
 	9385 3610 9525 3610
 $Comp
-L wat-rescue:C C9
+L digital-rescue:C-wat-rescue C9
 U 1 1 5FFFA89D
 P 2065 5465
@@
 $EndComp
 $Comp
-L wat-rescue:R R14
+L digital-rescue:R-wat-rescue R14
 U 1 1 5FFFA8B2
 P 2065 5025
@@
 	2065 4875 2065 4695
 $Comp
-L wat-rescue:C C10
+L digital-rescue:C-wat-rescue C10
 U 1 1 5FFFF00A
 P 3045 5465
@@
 $EndComp
 $Comp
-L wat-rescue:R R15
+L digital-rescue:R-wat-rescue R15
 U 1 1 5FFFF01F
 P 3045 5025
@@
 	3045 4875 3045 4695
 $Comp
-L wat-rescue:C C11
+L digital-rescue:C-wat-rescue C11
 U 1 1 6004F39B
 P 4020 5465
@@
 $EndComp
 $Comp
-L wat-rescue:R R16
+L digital-rescue:R-wat-rescue R16
 U 1 1 6004F3B0
 P 4020 5025
@@
 	4020 4875 4020 4695
 $Comp
-L wat-rescue:C C12
+L digital-rescue:C-wat-rescue C12
 U 1 1 6004F3BE
 P 5065 5465
@@
 $EndComp
 $Comp
-L wat-rescue:R R17
+L digital-rescue:R-wat-rescue R17
 U 1 1 6004F3D3
 P 5065 5025
@@
 	5065 4875 5065 4695
 $Comp
-L wat-rescue:C C13
+L digital-rescue:C-wat-rescue C13
 U 1 1 6004F3E1
 P 6190 5465
@@
 $EndComp
 $Comp
-L wat-rescue:R R18
+L digital-rescue:R-wat-rescue R18
 U 1 1 6004F3F6
 P 6190 5025
@@
 	6190 4875 6190 4695
 $Comp
-L wat-rescue:C C14
+L digital-rescue:C-wat-rescue C14
 U 1 1 60054BD1
 P 7280 5465
@@
 $EndComp
 $Comp
-L wat-rescue:R R19
+L digital-rescue:R-wat-rescue R19
 U 1 1 60054BE6
 P 7280 5025
@@
 	5505 4210 5510 4210
 $Comp
-L wat-rescue:NANO-nano Uxxx1
+L digital-rescue:NANO-nano-wat-rescue Uxxx1
 U 1 1 62EAD1BE
 P 6465 2045
@@
 jD8
 $Comp
-L wat-rescue:C C15
+L digital-rescue:C-wat-rescue C15
 U 1 1 6304975A
 P 8360 5465
@@
 $EndComp
 $Comp
-L wat-rescue:R R20
+L digital-rescue:R-wat-rescue R20
 U 1 1 63049766
 P 8360 5025
@@
 	8360 4875 8360 4695
 $Comp
-L wat-rescue:C C16
+L digital-rescue:C-wat-rescue C16
 U 1 1 63049771
 P 9485 5465
@@
 $EndComp
 $Comp
-L wat-rescue:R R21
+L digital-rescue:R-wat-rescue R21
 U 1 1 6304977D
 P 9485 5025
@@
 jD10
 $Comp
-L wat-rescue:C C17
+L digital-rescue:C-wat-rescue C17
 U 1 1 63098281
 P 10615 5465
@@
 $EndComp
 $Comp
-L wat-rescue:R R22
+L digital-rescue:R-wat-rescue R22
 U 1 1 6309828D
 P 10615 5025
@@
 	10615 4875 10615 4695
 $Comp
-L wat-rescue:C C18
+L digital-rescue:C-wat-rescue C18
 U 1 1 63098298
 P 1135 6920
@@
 $EndComp
 $Comp
-L wat-rescue:R R27
+L digital-rescue:R-wat-rescue R27
 U 1 1 630982A4
 P 1135 6480
@@
 	1135 6330 1135 6150
 $Comp
-L wat-rescue:C C19
+L digital-rescue:C-wat-rescue C19
 U 1 1 630982AF
 P 2215 6920
@@
 $EndComp
 $Comp
-L wat-rescue:R R28
+L digital-rescue:R-wat-rescue R28
 U 1 1 630982BB
 P 2215 6480
@@
 A2
 $Comp
-L wat-rescue:R R26
+L digital-rescue:R-wat-rescue R26
 U 1 1 635746A0
 P 3200 6475
@@
 	3200 6695 3455 6695
 $Comp
-L wat-rescue:R R25
+L digital-rescue:R-wat-rescue R25
 U 1 1 635746BC
 P 4125 6470
@@
 	4125 6320 4125 6140
 $Comp
-L wat-rescue:R R23
+L digital-rescue:R-wat-rescue R23
 U 1 1 635746D2
 P 5005 6465
@@
 	4125 6690 4380 6690
 $Comp
-L wat-rescue:R R24
+L digital-rescue:R-wat-rescue R24
 U 1 1 635746EF
 P 5925 6465
@@
 $Comp
 L ESP32_NODEMCU:ESP32_NODEMCU_OS U?
-U 1 1 6323ED7B
-P 12970 1930
-F 0 "U?" H 12970 3297 50  0000 C CNN
-F 1 "ESP32_NODEMCU_OS" H 12970 3206 50  0000 C CNN
-F 2 "MODULE_ESP32_NODEMCU" H 11140 2970 50  0001 L BNN
-F 3 "" H 12970 1930 50  0001 L BNN
-F 4 "Espressif" H 12970 1930 50  0001 L BNN "MANUFACTURER"
-F 5 "6.6 mm" H 11750 3300 50  0001 L BNN "MAXIMUM_PACKAGE_HEIGHT"
-F 6 "Manufacturer Recommendations" H 12540 3310 50  0001 L BNN "STANDARD"
-	1    12970 1930
-	1    0    0    -1
-$EndComp
+U 1 1 63250731
+P 12850 750
+F 0 "U?" H 12850 2117 50  0000 C CNN
+F 1 "ESP32_NODEMCU_OS" H 12850 2026 50  0000 C CNN
+F 2 "ESP32" H 12725 1700 50  0001 L BNN
+F 3 "" H 12850 750 50  0001 L BNN
+F 4 "Espressif" H 12675 1600 50  0001 L BNN "MANUFACTURER"
+F 5 "onsar" H 12725 1825 50  0001 L BNN "STANDARD"
+	1    12850 750
+	1    0    0    -1
+$EndComp

Commit message: trabajando en openControllerDigital
Parts:
- removed C10, C11, C12, C13, C14, C15, C16, C17, C18, C19, C3, C4, C5, C6, C7, C8, C9: 10nF, eco_power_v2:C_1206_HandSoldering, symbol digital-rescue:C-wat-rescue
- removed C2: 100nF, eco_power_v2:C_1206_HandSoldering, symbol digital-rescue:C-wat-rescue
- removed J4: e_i_02x10, symbol Connector_Generic:Conn_01x10
- removed R1, R10, R11, R12, R13, R14, R15, R16, R17, R18, R19, R2, R20, R21, R22, R23, R24, R25, R26, R27, R28, R3, R4, R5, R6, R7, R8, R9: 10k, eco_power_v2:R_1206_HandSoldering, symbol digital-rescue:R-wat-rescue
- removed Uxxx1: NANO-nano, MODULE, symbol digital-rescue:NANO-nano-wat-rescue
- added C10, C11, C12, C13, C14, C15, C16, C2, C3, C4, C5, C6, C7, C8, C9: 10nF, Capacitor_SMD:C_1206_3216Metric_Pad1.42x1.75mm_HandSolder, symbol digital-rescue:C-wat-rescue-digital-rescue
- added JP1: 23, Jumper:SolderJumper-2_P1.3mm_Open_RoundedPad1.0x1.5mm, symbol Jumper:SolderJumper_2_Open
- added JP2: 19, Jumper:SolderJumper-2_P1.3mm_Open_RoundedPad1.0x1.5mm, symbol Jumper:SolderJumper_2_Open
- added JP3: 18, Jumper:SolderJumper-2_P1.3mm_Open_RoundedPad1.0x1.5mm, symbol Jumper:SolderJumper_2_Open
- added JP4: 05, Jumper:SolderJumper-2_P1.3mm_Open_RoundedPad1.0x1.5mm, symbol Jumper:SolderJumper_2_Open
- added JP5: tx, Jumper:SolderJumper-2_P1.3mm_Open_RoundedPad1.0x1.5mm, symbol Jumper:SolderJumper_2_Open
- added JP6: rx, Jumper:SolderJumper-2_P1.3mm_Open_RoundedPad1.0x1.5mm, symbol Jumper:SolderJumper_2_Open
- added JP7: 04, Jumper:SolderJumper-2_P1.3mm_Open_RoundedPad1.0x1.5mm, symbol Jumper:SolderJumper_2_Open
- added R1, R19, R2, R20, R21, R22, R23, R24, R25, R26, R3, R4, R43, R5, R6: 4k7, Resistor_SMD:R_1206_3216Metric_Pad1.42x1.75mm_HandSolder, symbol digital-rescue:R-wat-rescue-digital-rescue
- added R10, R11, R12, R13, R14, R15, R16, R17, R18, R27, R28, R29, R30, R31, R32, R33, R34, R35, R36, R37, R38, R39, R40, R41, R42, R51, R59, R7, R8, R9: 10k, Resistor_SMD:R_1206_3216Metric_Pad1.42x1.75mm_HandSolder, symbol digital-rescue:R-wat-rescue-digital-rescue
- C1: value 10 -> 10nF; footprint (none) -> Capacitor_SMD:C_1206_3216Metric_Pad1.42x1.75mm_HandSolder
- D1: footprint (none) -> Digital:D_2114_3652Metric
- J1: footprint (none) -> Connector_Phoenix_MC:PhoenixContact_MCV_1,5_2-G-3.5_1x02_P3.50mm_Vertical
- J2: footprint (none) -> Connector_PinHeader_2.54mm:PinHeader_2x20_P2.54mm_Vertical
- J3: renamed from J5; footprint (none) -> Connector_Phoenix_MC:PhoenixContact_MCV_1,5_10-G-3.5_1x10_P3.50mm_Vertical
- J4: renamed from J3; footprint (none) -> Connector_Phoenix_MC:PhoenixContact_MCV_1,5_10-G-3.5_1x10_P3.50mm_Vertical
- U1: renamed from U?; footprint ESP32 -> Espressif:ESP32-DevKitC
Connections:
- net D2 is gone; now on net 3v3: J4.2 (Pin_2)
- net 5v_1: now also U1.19 (5V0), R1.2, R19.2, R2.2, R20.2, R21.2, R22.2, R23.2, R24.2, R25.2, R26.2, R3.2, R4.2, R43.2, R5.2, R6.2; no longer J3.10 (Pin_10), J3.5 (Pin_5)
- net D12: now also U1.13 (G12), R23.1, R31.1, R39.2
- net D13: now also U1.15 (G13), R24.1, R32.1, R40.2
- net GND: now also U1.14 (GND), U1.32 (GND), U1.38 (GND), C10.2, C11.2, C12.2, C13.2, C14.2, C15.2, C16.2, C2.2, C3.2, C4.2, C5.2, C6.2, C7.2, C8.2, C9.2, R13.1, R14.1, R15.1, R16.1, R17.1, R18.1, R35.1, R36.1, R37.1, R38.1, R39.1, R40.1, R41.1, R42.1, R59.1; no longer J2.23 (Pin_23), J2.24 (Pin_24), J2.26 (Pin_26), J2.40 (Pin_40), J3.6 (Pin_6)
- net SCL: now also U1.36 (SCL)
- net SDA: now also U1.33 (SDA)
- net RXD: now reaches J2.10 (Pin_10)
- net RXD: now also JP6.2 (B)
- net o04: now reaches J2.12 (Pin_12)
- net o04: now also JP7.2 (B)
- net o05: now reaches J2.15 (Pin_15)
- net o05: now also JP4.2 (B)
- net o18: now reaches J2.16 (Pin_16)
- net o18: now also JP3.2 (B)
- net o19: now reaches J2.18 (Pin_18)
- net o19: now also JP2.2 (B)
- net o23: now reaches J2.22 (Pin_22)
- net o23: now also JP1.2 (B)
- net TXD: now reaches J2.8 (Pin_8)
- net TXD: now also JP5.2 (B)
- net 3v3: now reaches U1.1 (3V3)
- net 3v3: now also J3.10 (Pin_10)
- net A26: now reaches U1.10 (G26)
- net A26: now also R20.1, R28.1, R36.2
- net D27: now reaches U1.11 (G27)
- net D27: now also R21.1, R29.1, R37.2
- net D14: now reaches U1.12 (G14)
- net D14: now also R22.1, R30.1, R38.2
- net D15: now reaches U1.23 (G15)
- net D15: now also R25.1, R33.1, R41.2
- net D02: now reaches U1.24 (G02)
- net D02: now also R26.1, R34.1, R42.2
- net D00: now reaches U1.25 (G00)
- net D00: now also R43.1, R51.1, R59.2
- net at U1.26 (G04): now also JP7.1 (A)
- net at U1.27 (G16): now also JP6.1 (A)
- net at U1.28 (G17): now also JP5.1 (A)
- net at U1.29 (G05): now also JP4.1 (A)
- net A36: now reaches U1.3 (G36)
- net A36: now also R1.1, R13.2, R7.1
- net at U1.30 (G18): now also JP3.1 (A)
- net at U1.31 (G19): now also JP2.1 (A)
- net at U1.37 (G23): now also JP1.1 (A)
- net A39: now reaches U1.4 (G39)
- net A39: now also R14.2, R2.1, R8.1
- net A34: now reaches U1.5 (G34)
- net A34: now also R15.2, R3.1, R9.1
- net A35: now reaches U1.6 (G35)
- net A35: now also R19.1, R27.1, R35.2
- net A32: now reaches U1.7 (G32)
- net A32: now also R10.1, R16.2, R4.1
- net A33: now reaches U1.8 (G33)
- net A33: now also R11.1, R17.2, R5.1
- net A25: now reaches U1.9 (G25)
- net A25: now also R12.1, R18.2, R6.1
- net D3 renamed jD27
- net jD27: now also C10.1, R29.2
- net D4 renamed jD14
- net jD14: now also C11.1, R30.2
- net D5 renamed jD12
- net jD12: now also C12.1, R31.2
- net D6 renamed jD13
- net jD13: now also C13.1, R32.2
- net D7 renamed jD15
- net jD15: now also C14.1, R33.2
- net D8 renamed jD02
- net jD02: now also C15.1, R34.2
- net D9 renamed jD00
- net jD00: now also C16.1, R51.2
- net jA0 renamed jA36
- net jA36: now also C2.1, R7.2
- net jA1 renamed jA39
- net jA39: now also C3.1, R8.2
- net jA2 renamed jA34
- net jA34: now also C4.1, R9.2
- net jA3 renamed jA33
- net jA33: now also C6.1, R11.2
- net jA6 renamed jA25
- net jA25: now also C7.1, R12.2
- net jA7 renamed jA26
- net jA26: now also C9.1, R28.2
- new net jA32: C5.1, J3.5 (Pin_5), R10.2
- new net jA35: C8.1, J3.6 (Pin_6), R27.2
- no-connect marks 33 -> 32
Other:
- moved on the sheet: C1, D1, J1, J2, J3, J4, U1

Commit message: ecotherm. actualizacion de los conectores phenix
Parts:
- J1: footprint Connector_Phoenix_MC:PhoenixContact_MCV_1,5_2-G-3.5_1x02_P3.50mm_Vertical -> Connector_Phoenix_MC:PhoenixContact_MC_1,5_2-G-3.5_1x02_P3.50mm_Horizontal
- J3, J4: footprint Connector_Phoenix_MC:PhoenixContact_MCV_1,5_10-G-3.5_1x10_P3.50mm_Vertical -> Connector_Phoenix_MC:PhoenixContact_MC_1,5_10-G-3.5_1x10_P3.50mm_Horizontal
Connections:
- net 3v3: now also J3.1 (Pin_1), J4.9 (Pin_9); no longer J3.10 (Pin_10), J4.2 (Pin_2)
- net 5v: now also J1.2 (Pin_2); no longer J1.1 (Pin_1)
- net 5v_1: now also J4.10 (Pin_10); no longer J4.1 (Pin_1)
- net GND: now also J1.1 (Pin_1), J3.10 (Pin_10), J4.1 (Pin_1); no longer J1.2 (Pin_2), J3.1 (Pin_1), J4.10 (Pin_10)
- net jA25: now also J3.8 (Pin_8); no longer J3.3 (Pin_3)
- net jA26: now also J3.9 (Pin_9); no longer J3.2 (Pin_2)
- net jA32: now also J3.6 (Pin_6); no longer J3.5 (Pin_5)
- net jA33: now also J3.7 (Pin_7); no longer J3.4 (Pin_4)
- net jA34: now also J3.4 (Pin_4); no longer J3.7 (Pin_7)
- net jA35: now also J3.5 (Pin_5); no longer J3.6 (Pin_6)
- net jA36: now also J3.2 (Pin_2); no longer J3.9 (Pin_9)
- net jA39: now also J3.3 (Pin_3); no longer J3.8 (Pin_8)
- net jD00: now also J4.2 (Pin_2); no longer J4.9 (Pin_9)
- net jD02: now also J4.3 (Pin_3); no longer J4.8 (Pin_8)
- net jD12: now also J4.6 (Pin_6); no longer J4.5 (Pin_5)
- net jD13: now also J4.5 (Pin_5); no longer J4.6 (Pin_6)
- net jD14: now also J4.7 (Pin_7); no longer J4.4 (Pin_4)
- net jD15: now also J4.4 (Pin_4); no longer J4.7 (Pin_7)
- net jD27: now also J4.8 (Pin_8); no longer J4.3 (Pin_3)
Changed lines of the file:
@@
 L Connector_Generic:Conn_01x02 J1
 U 1 1 622B6D5E
-P 1130 955
-F 0 "J1" H 1210 947 50  0000 L CNN
-F 1 "Conn_01x02" H 760 1145 50  0000 L CNN
-F 2 "Connector_Phoenix_MC:PhoenixContact_MCV_1,5_2-G-3.5_1x02_P3.50mm_Vertical" H 1130 955 50  0001 C CNN
-F 3 "~" H 1130 955 50  0001 C CNN
-	1    1130 955
-	1    0    0    -1
+P 1130 1055
+F 0 "J1" H 1210 1047 50  0000 L CNN
+F 1 "Conn_01x02" H 760 1245 50  0000 L CNN
+F 2 "Connector_Phoenix_MC:PhoenixContact_MC_1,5_2-G-3.5_1x02_P3.50mm_Horizontal" H 1130 1055 50  0001 C CNN
+F 3 "~" H 1130 1055 50  0001 C CNN
+	1    1130 1055
+	1    0    0    1
 $EndComp
 Text GLabel 930  955  0    50   Input ~ 0
@@
 F 0 "J4" H 7055 1842 50  0000 L CNN
 F 1 "e_i_01x10" H 6915 2380 50  0000 L CNN
-F 2 "Connector_Phoenix_MC:PhoenixContact_MCV_1,5_10-G-3.5_1x10_P3.50mm_Vertical" H 6975 1850 50  0001 C CNN
+F 2 "Connector_Phoenix_MC:PhoenixContact_MC_1,5_10-G-3.5_1x10_P3.50mm_Horizontal" H 6975 1850 50  0001 C CNN
 F 3 "~" H 6975 1850 50  0001 C CNN
 	1    6975 1850
 	1    0    0    -1
 $EndComp
-Text GLabel 6775 1450 0    50   Input ~ 0
-5v_1
-Text GLabel 6775 2350 0    50   Input ~ 0
-GND
-Text GLabel 6775 1550 0    50   Input ~ 0
+Text GLabel 5845 1750 0    50   Input ~ 0
+jA33
+Text GLabel 5845 1850 0    50   Input ~ 0
+jA32
+Text GLabel 5845 2250 0    50   Input ~ 0
+jA36
+Text GLabel 5845 2150 0    50   Input ~ 0
+jA39
+Text GLabel 5845 2050 0    50   Input ~ 0
+jA34
+Text GLabel 5845 1950 0    50   Input ~ 0
+jA35
+Text GLabel 5845 1650 0    50   Input ~ 0
+jA25
+Text GLabel 5845 1550 0    50   Input ~ 0
+jA26
+Text GLabel 5845 2350 0    50   Input ~ 0
 3v3
-Text GLabel 6775 1650 0    50   Input ~ 0
-jD27
-Text GLabel 6775 1750 0    50   Input ~ 0
-jD14
-Text GLabel 6775 1850 0    50   Input ~ 0
-jD12
-Text GLabel 6775 1950 0    50   Input ~ 0
-jD13
-Text GLabel 6775 2050 0    50   Input ~ 0
-jD15
-Text GLabel 6775 2150 0    50   Input ~ 0
-jD02
-Text GLabel 6775 2250 0    50   Input ~ 0
-jD00
-Text GLabel 5845 2050 0    50   Input ~ 0
-jA33
-Text GLabel 5845 1950 0    50   Input ~ 0
-jA32
-Text GLabel 5845 1550 0    50   Input ~ 0
-jA36
-Text GLabel 5845 1650 0    50   Input ~ 0
-jA39
-Text GLabel 5845 1750 0    50   Input ~ 0
-jA34
-Text GLabel 5845 1850 0    50   Input ~ 0
-jA35
-Text GLabel 5845 2150 0    50   Input ~ 0
-jA25
-Text GLabel 5845 2250 0    50   Input ~ 0
-jA26
 Text GLabel 5845 1450 0    50   Input ~ 0
-3v3
-Text GLabel 5845 2350 0    50   Input ~ 0
 GND
 $Comp
@@
 F 0 "J3" H 6125 1942 50  0000 L CNN
 F 1 "a_i_01x10" H 5995 2480 50  0000 L CNN
-F 2 "Connector_Phoenix_MC:PhoenixContact_MCV_1,5_10-G-3.5_1x10_P3.50mm_Vertical" H 6045 1950 50  0001 C CNN
+F 2 "Connector_Phoenix_MC:PhoenixContact_MC_1,5_10-G-3.5_1x10_P3.50mm_Horizontal" H 6045 1950 50  0001 C CNN
 F 3 "~" H 6045 1950 50  0001 C CNN
 	1    6045 1950
@@
 	1    0    0    -1
 $EndComp
+Text GLabel 6775 1550 0    50   Input ~ 0
+jD00
+Text GLabel 6775 1650 0    50   Input ~ 0
+jD02
+Text GLabel 6775 1750 0    50   Input ~ 0
+jD15
+Text GLabel 6775 1850 0    50   Input ~ 0
+jD13
+Text GLabel 6775 1950 0    50   Input ~ 0
+jD12
+Text GLabel 6775 2050 0    50   Input ~ 0
+jD14
+Text GLabel 6775 2150 0    50   Input ~ 0
+jD27
+Text GLabel 6775 2250 0    50   Input ~ 0
+3v3
+Text GLabel 6775 1450 0    50   Input ~ 0
+GND
+Text GLabel 6775 2350 0    50   Input ~ 0
+5v_1
 $EndSCHEMATC

Commit message: ecotherm. actualizacion del conector del bus
Parts:
- J2: footprint Connector_PinHeader_2.54mm:PinHeader_2x20_P2.54mm_Vertical -> Connector_PinSocket_2.54mm:PinSocket_2x20_P2.54mm_Vertical
Changed lines of the file:
@@
 F 0 "J2" H 3680 2897 50  0000 C CNN
 F 1 "Conn_02x20_Odd_Even" H 3680 2806 50  0000 C CNN
-F 2 "Connector_PinHeader_2.54mm:PinHeader_2x20_P2.54mm_Vertical" H 3630 1780 50  0001 C CNN
+F 2 "Connector_PinSocket_2.54mm:PinSocket_2x20_P2.54mm_Vertical" H 3630 1780 50  0001 C CNN
 F 3 "~" H 3630 1780 50  0001 C CNN
 	1    3630 1780
