File: open_controler_digital/digital/digital.kicad_pcb (KiCad board)
At the start: 2 copper layers, 56 x 85 mm, 84 parts, among them J1 d_o_01x10, J2 d_i_01x10, J3 Conn_02x20_Odd_Even, J4 Conn_01x02, Q1 BC856, Q10 JM, Q11 JM, Q12 JM, Q2 BC856, Q3 JM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

Commit message: digital. actualización de los conectores 3d
Parts:
- J1, J2: footprint Connector_Phoenix_MC:PhoenixContact_MCV_1,5_10-G-3.5_1x10_P3.50mm_Vertical -> Connector_Phoenix_MC:PhoenixContact_MC_1,5_10-G-3.5_1x10_P3.50mm_Horizontal
- J3: footprint Connector_PinHeader_2.54mm:PinHeader_2x20_P2.54mm_Vertical -> Connector_PinSocket_2.54mm:PinSocket_2x20_P2.54mm_Vertical; moved to B.Cu
- J4: footprint Connector_Phoenix_MC:PhoenixContact_MCV_1,5_2-G-3.5_1x02_P3.50mm_Vertical -> Connector_Phoenix_MC:PhoenixContact_MC_1,5_2-G-3.5_1x02_P3.50mm_Horizontal
- moved J1 31.5 mm to (75.7, 51.3), turned to 270 degrees
- moved J2 31.5 mm to (85.4, 124.2), turned to 0 degrees
- moved J4 3.50 mm to (75.5, 91.8), turned to 270 degrees
- turned J3 to 180 degrees
Connections:
- J1 pad 1: go1 -> vo0
- J1 pad 10: vo0 -> go1
- J1 pad 2: do12 -> do00
- J1 pad 3: do11 -> do01
- J1 pad 4: do10 -> do02
- J1 pad 5: vo1 -> go0
- J1 pad 6: go0 -> vo1
- J1 pad 7: do02 -> do10
- J1 pad 8: do01 -> do11
- J1 pad 9: do00 -> do12
- J2 pad 1: di20 -> GND_1
- J2 pad 10: GND_1 -> di20
- J2 pad 2: di21 -> 5v_1
- J2 pad 3: di22 -> gi3
- J2 pad 4: gi2 -> di32
- J2 pad 5: di30 -> di31
- J2 pad 6: di31 -> di30
- J2 pad 7: di32 -> gi2
- J2 pad 8: gi3 -> di22
- J2 pad 9: 5v_1 -> di21
- J4 pad 1: 5v -> GND_1
- J4 pad 2: GND_1 -> 5v
